File: hardware/v4/pi-parport.kicad_pcb (KiCad board)
At the start: 2 copper layers, 65 x 56 mm, 17 parts, among them J1 CONN_01X02, J2 40HAT, J3 Conn_02x13_Odd_Even, U1 CAT24C32, U2 SN74LVC161284DLR

Commit message: save work
Parts:
- removed J1: CONN_01X02, Connector_PinHeader_2.54mm:PinHeader_1x02_P2.54mm_Vertical
- removed R1: DNP, Resistor_SMD:R_0805_2012Metric_Pad1.15x1.40mm_HandSolder
- removed REF**: OSHW-Symbol_6.7x6mm_SilkScreen, Symbol:OSHW-Symbol_6.7x6mm_SilkScreen
- added C3: 100nF, Capacitor_SMD:C_0603_1608Metric_Pad1.08x0.95mm_HandSolder, F.Cu at (100.8, 75.2)
- added C4: 100nF, Capacitor_SMD:C_0603_1608Metric_Pad1.08x0.95mm_HandSolder, F.Cu at (100.8, 73.4)
- added C5: 100nF, Capacitor_SMD:C_0603_1608Metric_Pad1.08x0.95mm_HandSolder, F.Cu at (100.8, 71.6)
- added C6: 100nF, Capacitor_SMD:C_0603_1608Metric_Pad1.08x0.95mm_HandSolder, F.Cu at (100.8, 77.0)
- added H5: 3mm_Mounting_Hole, project_footprints:NPTH_3mm_ID, F.Cu at (140.0, 87.4)
- added H6: 3mm_Mounting_Hole, project_footprints:NPTH_3mm_ID, F.Cu at (82.0, 87.4)
- added J4: IEEE1284_DB25, Connector_Dsub:DSUB-25_Female_Horizontal_P2.77x2.84mm_EdgePinOffset7.70mm_Housed_MountingHolesOffset9.12mm, F.Cu at (127.4, 106.4)
- added J5: SERIAL0_DB9, Connector_Dsub:DSUB-9_Male_Horizontal_P2.77x2.84mm_EdgePinOffset7.70mm_Housed_MountingHolesOffset9.12mm, F.Cu at (89.3, 78.3)
- added J7: SERIAL0_IDC, Connector_PinHeader_2.54mm:PinHeader_2x05_P2.54mm_Vertical, F.Cu at (94.7, 69.6)
- added JP1: EEPROM WP, Jumper:SolderJumper-2_P1.3mm_Open_RoundedPad1.0x1.5mm, B.Cu at (135.7, 71.9)
- added JP2: DTR+RTS, Jumper:SolderJumper-2_P1.3mm_Open_RoundedPad1.0x1.5mm, B.Cu at (95.4, 83.1)
- added JP3: DSR+CTS, Jumper:SolderJumper-2_P1.3mm_Open_RoundedPad1.0x1.5mm, B.Cu at (95.4, 87.6)
- added JP4: TX_SEL, Jumper:SolderJumper-3_P1.3mm_Bridged12_RoundedPad1.0x1.5mm, B.Cu at (100.3, 82.5)
- added JP5: RTS_SEL, Jumper:SolderJumper-3_P1.3mm_Bridged12_RoundedPad1.0x1.5mm, B.Cu at (105.4, 82.5)
- added JP6: RX_SEL, Jumper:SolderJumper-3_P1.3mm_Bridged12_RoundedPad1.0x1.5mm, B.Cu at (102.9, 82.5)
- added JP7: CTS_SEL, Jumper:SolderJumper-3_P1.3mm_Bridged12_RoundedPad1.0x1.5mm, B.Cu at (108.0, 82.5)
- added U3: MAX3232, Package_SO:SO-16_3.9x9.9mm_P1.27mm, F.Cu at (106.4, 74.9)
- C1, C2: footprint Capacitor_SMD:C_0805_2012Metric_Pad1.15x1.40mm_HandSolder -> Capacitor_SMD:C_0603_1608Metric_Pad1.08x0.95mm_HandSolder
- J3: value Conn_02x13_Odd_Even -> IEEE1284_IDC; footprint Connector_PinHeader_2.54mm:PinHeader_2x13_P2.54mm_Horizontal -> Connector_PinHeader_2.54mm:PinHeader_2x13_P2.54mm_Vertical
- R2, R3, R4, R5: footprint Resistor_SMD:R_0805_2012Metric_Pad1.15x1.40mm_HandSolder -> Resistor_SMD:R_0603_1608Metric_Pad0.98x0.95mm_HandSolder
- moved J3 46.3 mm to (134.4, 86.9), turned to -90 degrees
- moved U1 44.6 mm to (135.7, 72.0)
- moved R3 42.8 mm to (141.3, 74.9)
- moved R4 42.2 mm to (141.3, 73.2)
- moved R2 42.1 mm to (141.3, 71.4)
- moved C1 39.2 mm to (114.3, 69.5), turned to 0 degrees
- moved U2 11.5 mm to (123.7, 75.7), turned to 0 degrees
- moved C2 11.1 mm to (130.0, 74.8)
- moved R5 10.9 mm to (116.3, 82.7)
Connections:
- J2 pad 10: Net-(J2-Pad10) -> UART_RX
- J2 pad 11: /GPIO17 -> UART_RTS
- J2 pad 13: Net-(J2-Pad13) -> /GPIO27
- J2 pad 17: Net-(J2-Pad17) -> unconnected-(J2-P3V3-Pad17)
- J2 pad 26: Net-(J2-Pad26) -> unconnected-(J2-BCM7-Pad26)
- J2 pad 29: Net-(J2-Pad29) -> unconnected-(J2-BCM5-Pad29)
- J2 pad 32: Net-(J2-Pad32) -> unconnected-(J2-BCM12-Pad32)
- J2 pad 36: Net-(J2-Pad36) -> UART_CTS
- J2 pad 8: Net-(J2-Pad8) -> UART_TX
- J3 pad 10: GND -> /STATUS6
- J3 pad 11: /DATA4 -> /STATUS7
- J3 pad 12: GND -> /STATUS5
- J3 pad 13: /DATA5 -> /STATUS4
- J3 pad 14: GND -> /CONTROL1
- J3 pad 15: /DATA6 -> /STATUS3
- J3 pad 16: GND -> /CONTROL2
- J3 pad 17: /DATA7 -> /CONTROL3
- J3 pad 19: /STATUS6 -> GND
- J3 pad 2: /CONTROL1 -> /DATA0
- J3 pad 21: /STATUS7 -> GND
- J3 pad 23: /STATUS5 -> GND
- J3 pad 25: /STATUS4 -> GND
- J3 pad 3: /DATA0 -> /DATA1
- J3 pad 4: /STATUS3 -> /DATA2
- J3 pad 5: /DATA1 -> /DATA3
- J3 pad 6: /CONTROL2 -> /DATA4
- J3 pad 7: /DATA2 -> /DATA5
- J3 pad 8: /CONTROL3 -> /DATA6
- J3 pad 9: /DATA3 -> /DATA7
- U2 pad 20: /GPIO17 -> /GPIO27
- U2 pad 30: Net-(U2-Pad30) -> unconnected-(U2-PERI_OUT-Pad30)
- U2 pad 43: Net-(U2-Pad43) -> unconnected-(U2-Y13-Pad43)
Routing:
- net +5V: track 59.9 -> 0.00 mm
- net /ID_SC_EEPROM: track 86.2 -> 28.4 mm, vias 1 -> 2
- net /ID_SD_EEPROM: track 84.9 -> 27.9 mm
- net CTS: track 0.00 -> 48.8 mm
- net DSR: track 0.00 -> 42.0 mm
- net RTS: track 0.00 -> 39.4 mm, vias 0 -> 2
- net UART_CTS: track 0.00 -> 38.1 mm, vias 0 -> 1
- net DTR: track 0.00 -> 34.5 mm
- net RX: track 0.00 -> 33.2 mm, vias 0 -> 1
- net UART_TX: track 0.00 -> 32.0 mm, vias 0 -> 1
- net GND: track 29.7 -> 0.00 mm, vias 27 -> 0
- net TX: track 0.00 -> 28.7 mm, vias 0 -> 1
- net /GPIO27: track 0.00 -> 28.3 mm, vias 0 -> 1
- net /STATUS4: track 34.8 -> 62.8 mm, vias 0 -> 1
- net UART_RTS: track 0.00 -> 27.0 mm, vias 0 -> 1
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Other:
- outline, holes or cut-outs redrawn
- net class Default removed
- board text added: "1:1 DB9M"
- board text added: "Null-Modem DB9F"
